File: B0_DC12_DC51.1.brd (EAGLE design)
At the start: 36 parts, among them Q1 BD140, Q2 BD139, Q3 BD140, Q4 BD139, X1 5566-24, X2 5566-6

Commit message: .
Parts:
- added JP1: (no value), Разъёмы штырьковые 2.54мм:1X01
- added U$1: (no value), h:H44X32
- Q1, Q3: value BD140 -> (none); device transistor-pnp:TO126 -> transistor:TO126V
- Q2, Q4: value BD139 -> (none); device transistor-npn:TO126 -> transistor:TO126V
- moved Q2 6.84 mm to (-76.2, -3.81), turned to 270 degrees
- moved R6 6.63 mm to (-62.2, 12.1), turned to 180 degrees
- moved Q1 6.35 mm to (-71.1, -3.81), turned to 270 degrees
- moved R7 5.72 mm to (-58.4, 8.26)
- moved R8 4.45 mm to (-63.5, 4.45)
- moved DA3 4.26 mm to (-58.4, -5.71), turned to 90 degrees
- moved Q3 3.42 mm to (-74.3, -14.0), turned to 90 degrees
- moved Q4 1.27 mm to (-78.7, -14.0), turned to 90 degrees
Routing:
- net GND: track 49.0 -> 66.1 mm
- net N$11: track 15.4 -> 4.44 mm
- net N$10: track 13.8 -> 4.44 mm
- net N$9: track 13.8 -> 5.08 mm
- net N$8: track 12.0 -> 5.08 mm
- net N$15: track 15.2 -> 17.8 mm

Commit message: .
Parts:
- removed Q2: (no value), transistor:TO126V
- removed R11: 470, rcl:0207/12
- removed R12: 15k, rcl:0207/12
- added R15, R16: 470, rcl:M0805
- added R17, R18, R19: 22, rcl:M0805
- added VT10, VT12, VT9: (no value), m_transistor:DPACK
- R1: value 10k -> 15k; device rcl:0207/12 -> rcl:M0805
- R10: value 100k -> 3k3
- R13: value 220 -> 39; device rcl:0207/12 -> rcl:M0805
- R14: value 10k -> 39
- R2: value 22 -> 470
- R3: value 22 -> 100k; device rcl:M0805 -> rcl:R0805
- R4: value 22 -> 220
- R6: value 470 -> 10k; device rcl:M0805 -> rcl:0207/12
- R7: value 39 -> 10k
- R8: value 470 -> 3k3; device rcl:M0805 -> rcl:0207/12
- R9: value 39 -> 1k; device rcl:M0805 -> rcl:0207/12
- VT1: value (none) -> 2N5401; device m_transistor:DPACK -> m_transistor:TO92
- VT2: value (none) -> 2N5551; device m_transistor:DPACK -> m_transistor:TO92
- VT4: device m_transistor:DPACK -> transistor:TO126V
- moved R8 149.7 mm to (-121.9, -133.3), flipped to the top, turned to 0 degrees
- moved R7 135.6 mm to (-109.2, -117.5), flipped to the top
- moved R9 130.1 mm to (-121.9, -128.9), flipped to the top
- moved R14 114.2 mm to (-61.0, -14.0), flipped to the bottom
- moved R13 111.4 mm to (-58.4, 8.26), flipped to the bottom
- moved R10 77.0 mm to (-121.9, -137.8)
- moved R4 76.1 mm to (-104.1, -93.3), flipped to the top
- moved R2 71.9 mm to (-104.1, -73.7), flipped to the top
- moved R6 64.1 mm to (-80.0, -49.5), flipped to the top, turned to 0 degrees
- moved R3 51.9 mm to (-94.0, -52.7), flipped to the top
- moved VT1 48.9 mm to (-112.4, -43.8), flipped to the top
- moved R1 46.2 mm to (-104.1, -88.9)
- moved VT2 39.2 mm to (-112.4, -36.2), flipped to the top
- moved VT4 21.8 mm to (-76.2, -3.81), flipped to the top, turned to 270 degrees
- renumbered Q1 to VT5, Q3 to VT7, Q4 to VT6, R5 to R20, VT3 to VT11
Connections:
- new net N$23: R10.2, R9.1, VT1.3
- new net N$24: R9.2, VT1.1
- new net N$25: R8.2, VT1.2
- new net N$26: R10.1, VT2.2
- net GND: now also R15.1, R16.1, VT10.S, VT12.S, VT9.S; no longer R12.1, VT1.S, VT2.S, VT4.S
- net N$1: now also R6.2; no longer R1.2
- net N$10: now also R14.2, R16.2; no longer R8.2, R9.2
- net N$11: now also R19.1; no longer R4.1
- net N$12: now also VT12.D; no longer VT4.D
- net N$13: now also R13.1; no longer R7.1
- net N$14: now also R14.1; no longer R9.1
- net N$15: now also VT4.2; no longer Q2.2
- net N$16: now also R7.2; no longer R14.2
- net N$17: now also R19.2; no longer R4.2
- net N$18: now also VT12.G; no longer VT4.G
- net N$19: now also R1.2, R4.1; no longer R12.2, R13.1
- net N$22: now also R2.2, R3.2; no longer R10.2, R11.2
- net N$3: now also VT10.D, VT9.D; no longer VT1.D, VT2.D
- net N$4: now also R17.2, VT9.G; no longer R2.2, VT1.G
- net N$5: now also R18.2, VT10.G; no longer R3.2, VT2.G
- net N$6: now also R3.1; no longer R10.1
- net N$7: now also R2.1, R7.1; no longer R11.1, R14.1
- net N$8: now also R13.2, R15.2, VT4.3; no longer Q2.3, R6.2, R7.2
- net N$9: now also R17.1, R18.1, VT4.1; no longer Q2.1, R2.1, R3.1

Commit message: .
Parts:
- added C10: 100n, rcl:C0805
- added C20: 407n, rcl:C0805
- added C9: 220n, rcl:C0805
- added OK1: PC817, optocoupler:DIL04
- added R11: 100k, rcl:M0805
- added R12: 10k, rcl:M0805
- added R21: 6k8, rcl:M0805
- added R22: 33k, rcl:M0805
- added R23: 3k3, rcl:M0805
- added R24: 220, rcl:M0805
- added R25: 2k, rcl:M0805
- added R26: 10k, rcl:RTRIM3296W
- added R33: 100k, rcl:RTRIM3296W
- added R34: 22k, rcl:M0805
- added R37: 47k, rcl:M0805
- added VD4: (no value), diode:DO41-7.6
- added VT3, VT8: 2N5551, m_transistor:TO92
- R10, R8, R9: device rcl:0207/12 -> rcl:M0805
- moved JP1 172.4 mm to (-21.6, 11.4)
- moved R10 169.6 mm to (-22.2, -0.64), flipped to the bottom, turned to 90 degrees
- moved R9 166.4 mm to (-28.6, 8.89), flipped to the bottom
- moved R8 164.3 mm to (-28.6, 1.91), flipped to the bottom, turned to 90 degrees
- moved X1 142.8 mm to (-111.8, 34.9)
- moved X2 142.8 mm to (-59.7, 34.9)
- moved X3 142.8 mm to (-129.5, 19.7)
- moved D3 107.5 mm to (-41.9, -29.2), flipped to the bottom, turned to 90 degrees
- moved R7 99.9 mm to (-55.9, -33.0), flipped to the bottom
- moved VT1 98.0 mm to (-28.6, 6.99)
- moved D2 95.8 mm to (-49.5, -33.7), flipped to the bottom
- moved VT2 89.0 mm to (-28.6, -6.35), turned to 180 degrees
- moved R4 86.9 mm to (-47.6, -27.3), flipped to the bottom, turned to 270 degrees
- moved R1 81.4 mm to (-54.0, -24.8), flipped to the bottom, turned to 180 degrees
- moved C6 77.5 mm to (-59.1, -23.5), flipped to the bottom
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Connections:
- net N$13 renamed CL13
- net N$14 renamed CL14
- removed net N$16: C3.1, C7.-, DA3.13, DA3.14, R7.2
- removed net N$25: R8.2, VT1.2
- new net +12V: R21.2
- new net +5VREF: C3.1, C7.-, DA3.13, DA3.14, OK1.4, R12.2, R7.2, R9.2, VT1.1
- new net N$13: D3.A, DA3.16, R8.2, VT1.2
- new net N$14: OK1.3, R4.2
- new net N$27: R12.1, VT2.3, VT3.2
- new net N$28: R11.2, VT2.1, VT3.1
- new net N$29: R22.1, R23.2, VT3.3, VT8.2
- new net N$30: C9.1, R21.1, R22.2
- new net N$31: R24.1, VT8.3
- new net N$32: C10.2, R24.2, R25.2, VD4.C
- new net N$33: R26.2, VD4.A
- new net N$34: R26.1
- new net V+: C20.1, OK1.1, R34.2
- new net V-: R37.2
- net GND: now also C10.1, C9.2, R11.1, R23.1, R25.1, R26.3, VT8.1
- net N$21: now also C20.2, OK1.2, R33.1, R33.2, R37.1; no longer D3.A, DA3.16
- net N$24: now also R33.3, R34.1; no longer R9.2, VT1.1

Commit message: .
Parts:
- added D4, D6: (no value), diode:SOT93L
- moved R37 124.4 mm to (-81.9, -40.0), flipped to the bottom, turned to 270 degrees
- moved R34 113.5 mm to (-94.0, -31.8), flipped to the bottom, turned to 180 degrees
- moved R33 112.2 mm to (-91.4, -29.2), turned to 90 degrees
- moved C20 111.7 mm to (-85.1, -31.1), flipped to the bottom, turned to 270 degrees
- moved OK1 106.8 mm to (-85.1, -31.1), turned to 270 degrees
- moved R6 72.3 mm to (-52.1, 17.1), turned to 270 degrees
- moved C4 70.9 mm to (-54.6, 10.8), turned to 90 degrees
- moved R7 42.2 mm to (-40.6, 6.35), turned to 90 degrees
- moved D2 33.9 mm to (-39.4, -1.27)
- moved D3 31.2 mm to (-43.8, 1.91), turned to 180 degrees
- moved R15 20.7 mm to (-48.3, 15.9), turned to 180 degrees
- moved R13 19.3 mm to (-43.8, 15.9)
- moved D1 17.1 mm to (-50.2, -5.08)
- moved C5 17.1 mm to (-54.6, 6.35)
- moved DA3 17.1 mm to (-46.4, 8.89)
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Routing:
- net GND: track 66.1 -> 65.5 mm

Commit message: .
Parts:
- removed D4, D6: (no value), diode:SOT93L
- added VD1: 2v4, diode:SOD80C
- added VD2: 4148, diode:SOD80C
- C2: value 470x25v -> 47n; device rcl:E5-10,5 -> rcl:C0805
- C3: value 470n -> 820; device rcl:C0805 -> rcl:C025-025X050
- C4: value 820 -> 220n; device rcl:C025-025X050 -> rcl:C0805
- C5: value 47n -> 470x25v; device rcl:C0805 -> rcl:E5-10,5
- C6: value 220n -> 47x25v; device rcl:C0805 -> rcl:E5-10,5
- C7: value 47x25v -> 470n; device rcl:E5-10,5 -> rcl:C0805
- D1, D2: value (none) -> SBL4020; device diode:SOD80C -> diodes:TO247H
- VD3: value (none) -> 4148
- moved D1 95.1 mm to (-130.2, -56.5), flipped to the top
- moved D2 85.0 mm to (-102.2, -58.4), flipped to the top
- moved C3 56.6 mm to (-54.6, 10.8), flipped to the top, turned to 90 degrees
- moved C2 40.6 mm to (-54.6, 6.35), flipped to the bottom, turned to 90 degrees
- moved C5 40.6 mm to (-68.6, -31.8), flipped to the top, turned to 0 degrees
- moved C4 37.4 mm to (-67.9, -24.1), flipped to the bottom, turned to 180 degrees
- moved C6 32.7 mm to (-59.7, -45.1), flipped to the top, turned to 90 degrees
- moved C7 17.6 mm to (-76.8, -41.3), flipped to the bottom, turned to 0 degrees
- moved C1 17.1 mm to (-55.2, -12.7), turned to 0 degrees
- renumbered D3 to VD3
Connections:
- net +5VREF: now also C6.-, C7.1; no longer C3.1, C7.-
- net GND: now also C5.-, C7.2, VD1.A, VD2.A; no longer C2.-, C6.2, D1.A, D2.A
- net N$15: now also C4.1, C5.+; no longer C1.1, C2.+
- net N$2: now also C3.1; no longer C4.1
- net N$20: now also C6.+, VD2.C; no longer C7.+, D2.C
- net N$22: now also C2.1; no longer C5.1
- net N$6: now also C2.2; no longer C5.2
- net N$7: now also C1.1, VD1.C; no longer C6.1, D1.C
Changed lines of the file:
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@@
 <dimension x1="-86.36" y1="41.275" x2="-66.04" y2="42.545" x3="-76.2" y3="46.99" textsize="1.778" layer="21" dtype="horizontal"/>
 <dimension x1="-145.415" y1="-53.34" x2="-44.45" y2="-57.785" x3="-94.9325" y3="57.785" textsize="1.778" layer="21" dtype="horizontal"/>
-<circle x="-124.46" y="-5.715" radius="20" width="1.016" layer="21"/>
+<circle x="-125.095" y="-5.715" radius="20" width="1.016" layer="21"/>
 <circle x="-141.605" y="31.75" radius="3" width="0.5" layer="21"/>
 <circle x="-48.26" y="31.75" radius="3" width="0.5" layer="21"/>
@@
 <element name="R16" library="rcl" package="M0805" value="470" x="-59.055" y="1.27" rot="MR180"/>
 <element name="R14" library="rcl" package="M0805" value="39" x="-52.07" y="0.635" rot="MR0"/>
-<element name="C1" library="rcl" package="C0805" value="220n" x="-67.945" y="-24.13" rot="MR180"/>
-<element name="C2" library="rcl" package="E5-10,5" value="470x25v" x="-68.58" y="-31.75"/>
-<element name="C3" library="rcl" package="C0805" value="470n" x="-76.835" y="-41.275" rot="MR0"/>
+<element name="C4" library="rcl" package="C0805" value="220n" x="-67.945" y="-24.13" rot="MR180"/>
+<element name="C5" library="rcl" package="E5-10,5" value="470x25v" x="-68.58" y="-31.75"/>
+<element name="C7" library="rcl" package="C0805" value="470n" x="-76.835" y="-41.275" rot="MR0"/>
 <element name="R6" library="rcl" package="0207/12" value="10k" x="-52.07" y="17.145" rot="R270"/>
-<element name="C4" library="rcl" package="C025-025X050" value="820" x="-54.61" y="10.795" rot="R90"/>
+<element name="C3" library="rcl" package="C025-025X050" value="820" x="-54.61" y="10.795" rot="R90"/>
 <element name="VT9" library="m_transistor" package="DPACK" value="" x="-84.455" y="3.81" rot="MR0"/>
 <element name="VT10" library="m_transistor" package="DPACK" value="" x="-92.075" y="3.81" rot="MR0"/>
@@
 <element name="R20" library="rcl" package="M0805" value="22" x="-78.74" y="-19.05" rot="MR0"/>
 <element name="R3" library="rcl" package="R0805" value="100k" x="-52.07" y="6.35" rot="MR270"/>
-<element name="C5" library="rcl" package="C0805" value="47n" x="-54.61" y="6.35" rot="MR90"/>
+<element name="C2" library="rcl" package="C0805" value="47n" x="-54.61" y="6.35" rot="MR90"/>
 <element name="R2" library="rcl" package="M0805" value="470" x="-46.355" y="-1.27" rot="MR0"/>
-<element name="D1" library="diode" package="SOD80C" value="" x="-50.165" y="-5.08" rot="MR0"/>
-<element name="C6" library="rcl" package="C0805" value="220n" x="-55.245" y="-12.7" rot="MR0"/>
+<element name="VD1" library="diode" package="SOD80C" value="2v4" x="-50.165" y="-5.08" rot="MR0"/>
+<element name="C1" library="rcl" package="C0805" value="220n" x="-55.245" y="-12.7" rot="MR0"/>
 <element name="R1" library="rcl" package="M0805" value="15k" x="-49.53" y="-12.065" rot="MR180"/>
 <element name="R4" library="rcl" package="M0805" value="220" x="-45.72" y="-15.24" rot="MR270"/>
-<element name="C7" library="rcl" package="E5-10,5" value="47x25v" x="-59.69" y="-45.085" rot="R90"/>
-<element name="D2" library="diode" package="SOD80C" value="" x="-39.37" y="-1.27" rot="MR0"/>
-<element name="D3" library="diode" package="SOD80C" value="" x="-43.815" y="1.905" rot="MR180"/>
+<element name="C6" library="rcl" package="E5-10,5" value="47x25v" x="-59.69" y="-45.085" rot="R90"/>
+<element name="VD2" library="diode" package="SOD80C" value="4148" x="-39.37" y="-1.27" rot="MR0"/>
+<element name="VD3" library="diode" package="SOD80C" value="4148" x="-43.815" y="1.905" rot="MR180"/>
 <element name="R7" library="rcl" package="M0805" value="10k" x="-40.64" y="6.35" rot="MR90"/>
 <element name="U$1" library="h" package="H44X32" value="" x="-87.63" y="-6.985" rot="R90"/>
@@
 <element name="R34" library="rcl" package="M0805" value="22k" x="-93.98" y="-31.75" rot="MR180"/>
 <element name="R37" library="rcl" package="M0805" value="47k" x="-81.915" y="-40.005" rot="MR270"/>
-<element name="D4" library="diode" package="SOT93L" value="" x="-111.125" y="-26.035"/>
-<element name="D6" library="diode" package="SOT93L" value="" x="-137.16" y="-29.21"/>
+<element name="D1" library="diodes" package="TO247H" value="SBL4020" x="-130.175" y="-56.515"/>
+<element name="D2" library="diodes" package="TO247H" value="SBL4020" x="-102.235" y="-58.42"/>
 </elements>
 <signals>
@@
 <contactref element="R16" pad="1"/>
 <contactref element="DA3" pad="7"/>
-<contactref element="C1" pad="2"/>
-<contactref element="C2" pad="-"/>
-<contactref element="C3" pad="2"/>
+<contactref element="C4" pad="2"/>
+<contactref element="C5" pad="-"/>
+<contactref element="C7" pad="2"/>
 <contactref element="R6" pad="1"/>
 <contactref element="VT10" pad="S"/>
@@
 <wire x1="-97.79" y1="-18.77" x2="-97.79" y2="-3.81" width="1.016" layer="16"/>
 <wire x1="-97.79" y1="-3.81" x2="-94.355" y2="-3.81" width="1.016" layer="16"/>
-<contactref element="D1" pad="A"/>
-<contactref element="C6" pad="2"/>
+<contactref element="VD1" pad="A"/>
+<contactref element="C1" pad="2"/>
 <contactref element="R1" pad="1"/>
-<contactref element="D2" pad="A"/>
+<contactref element="VD2" pad="A"/>
 <wire x1="-63.5" y1="-1.27" x2="-60.325" y2="-1.27" width="1.016" layer="16"/>
 <wire x1="-60.325" y1="-1.27" x2="-60.325" y2="-11.43" width="1.016" layer="16"/>
@@
 <contactref element="C9" pad="2"/>
 <contactref element="R26" pad="3"/>
-<contactref element="C4" pad="2"/>
+<contactref element="C3" pad="2"/>
 <wire x1="-66.04" y1="-31.75" x2="-77.785" y2="-41.275" width="0" layer="19" extent="16-16"/>
 <wire x1="-66.995" y1="-24.13" x2="-66.04" y2="-31.75" width="0" layer="19" extent="16-16"/>
@@
 <contactref element="VT6" pad="2"/>
 <contactref element="VT4" pad="2"/>
-<contactref element="C1" pad="1"/>
-<contactref element="C2" pad="+"/>
+<contactref element="C4" pad="1"/>
+<contactref element="C5" pad="+"/>
 <wire x1="-68.58" y1="-1.27" x2="-72.39" y2="-1.27" width="1.016" layer="16"/>
 <wire x1="-72.39" y1="-1.27" x2="-72.39" y2="-11.43" width="1.016" layer="16"/>
@@
 <signal name="N$2">
 <contactref element="DA3" pad="5"/>
-<contactref element="C4" pad="1"/>
+<contactref element="C3" pad="1"/>
 <wire x1="-49.4284" y1="9.525" x2="-54.61" y2="9.525" width="0" layer="19" extent="16-16"/>
 </signal>
@@
 <contactref element="DA3" pad="3"/>
 <contactref element="R3" pad="1"/>
-<contactref element="C5" pad="2"/>
+<contactref element="C2" pad="2"/>
 <wire x1="-52.07" y1="7.3" x2="-54.61" y2="7.3" width="0" layer="19" extent="16-16"/>
 <wire x1="-49.4284" y1="6.985" x2="-52.07" y2="7.3" width="0" layer="19" extent="16-16"/>
@@
 <contactref element="DA3" pad="2"/>
 <contactref element="R3" pad="2"/>
-<contactref element="C5" pad="1"/>
+<contactref element="C2" pad="1"/>
 <contactref element="R2" pad="2"/>
 <wire x1="-52.07" y1="5.4" x2="-54.61" y2="5.4" width="0" layer="19" extent="16-16"/>
@@
 <contactref element="DA3" pad="15"/>
 <contactref element="R2" pad="1"/>
-<contactref element="D1" pad="C"/>
-<contactref element="C6" pad="1"/>
+<contactref element="VD1" pad="C"/>
+<contactref element="C1" pad="1"/>
 <contactref element="R7" pad="1"/>
 <wire x1="-48.465" y1="-5.08" x2="-54.295" y2="-12.7" width="0" layer="19" extent="16-16"/>
@@
 </signal>
 <signal name="N$20">
-<contactref element="C7" pad="+"/>
+<contactref element="C6" pad="+"/>
 <contactref element="DA3" pad="4"/>
-<contactref element="D2" pad="C"/>
-<contactref element="D3" pad="C"/>
+<contactref element="VD2" pad="C"/>
+<contactref element="VD3" pad="C"/>
 <wire x1="-37.67" y1="-1.27" x2="-59.69" y2="-47.625" width="0" layer="19" extent="16-16"/>
 <wire x1="-45.515" y1="1.905" x2="-37.67" y2="-1.27" width="0" layer="19" extent="16-16"/>
@@
 <contactref element="DA3" pad="13"/>
 <contactref element="DA3" pad="14"/>
-<contactref element="C3" pad="1"/>
-<contactref element="C7" pad="-"/>
+<contactref element="C7" pad="1"/>
+<contactref element="C6" pad="-"/>
 <contactref element="VT1" pad="1"/>
 <contactref element="R9" pad="2"/>
@@
 <contactref element="R8" pad="2"/>
 <contactref element="VT1" pad="2"/>
+<contactref element="VD3" pad="A"/>
 <contactref element="DA3" pad="16"/>
-<contactref element="D3" pad="A"/>
-<wire x1="-42.115" y1="1.905" x2="-43.2816" y2="4.445" width="0" layer="19" extent="16-16"/>
+<wire x1="-43.2816" y1="4.445" x2="-42.115" y2="1.905" width="0" layer="19" extent="16-16"/>
 <wire x1="-19.685" y1="5.395" x2="-42.115" y2="1.905" width="0" layer="19" extent="16-16"/>
 <wire x1="-19.685" y1="8.255" x2="-19.685" y2="5.395" width="0" layer="19" extent="16-16"/>
