File: B0_DC12_DC51.1.brd (EAGLE design)
At the start: 63 parts, among them X1 5566-24, X2 5566-6

Commit message: 2
Parts:
- added R27: 240, rcl:0207/10
- added TV1B: (no value), Разъёмы штырьковые 2.54мм:1X03
- added VD5, VD6: 4148, diode:SOD80C
- moved D2 2.29 mm to (-103.5, -56.5)
Connections:
- new net N$16: R27.2, TV1B.1, VD5.A
- new net N$25: R27.1, TV1B.3, VD6.A
- net GND: now also TV1B.2
- net N$34: now also VD5.C, VD6.C
Changed lines of the file:
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@@
 <element name="R37" library="rcl" package="M0805" value="47k" x="-81.915" y="-40.005" rot="MR270"/>
 <element name="D1" library="diodes" package="TO247H" value="SBL4020" x="-130.175" y="-56.515"/>
-<element name="D2" library="diodes" package="TO247H" value="SBL4020" x="-102.235" y="-58.42"/>
+<element name="D2" library="diodes" package="TO247H" value="SBL4020" x="-103.505" y="-56.515"/>
+<element name="TV1B" library="Разъёмы штырьковые 2.54мм" package="1X03" value="" x="-161.925" y="-14.605"/>
+<element name="VD5" library="diode" package="SOD80C" value="4148" x="-164.465" y="-8.89" rot="MR270"/>
+<element name="VD6" library="diode" package="SOD80C" value="4148" x="-159.385" y="-8.89" rot="MR270"/>
+<element name="R27" library="rcl" package="0207/10" value="240" x="-161.925" y="-17.78" rot="R180"/>
 </elements>
 <signals>
@@
 <contactref element="R26" pad="3"/>
 <contactref element="C3" pad="2"/>
-<wire x1="-66.04" y1="-31.75" x2="-77.785" y2="-41.275" width="0" layer="19" extent="16-16"/>
-<wire x1="-66.995" y1="-24.13" x2="-66.04" y2="-31.75" width="0" layer="19" extent="16-16"/>
+<contactref element="TV1B" pad="2"/>
+<wire x1="-97.79" y1="-18.77" x2="-161.925" y2="-14.605" width="0" layer="19" extent="16-16"/>
+<wire x1="-66.995" y1="-24.13" x2="-87.37" y2="-22.225" width="0" layer="19" extent="16-16"/>
+<wire x1="-66.04" y1="-31.75" x2="-66.995" y2="-24.13" width="0" layer="19" extent="16-16"/>
 <wire x1="-64.135" y1="-11.43" x2="-66.995" y2="-24.13" width="0" layer="19" extent="16-16"/>
 <wire x1="-60.005" y1="1.27" x2="-60.325" y2="-1.27" width="0" layer="19" extent="16-16"/>
@@
 <wire x1="-49.21" y1="15.875" x2="-49.4284" y2="12.065" width="0" layer="19" extent="16-16"/>
 <wire x1="-52.07" y1="23.495" x2="-49.21" y2="15.875" width="0" layer="19" extent="16-16"/>
+<wire x1="-77.785" y1="-41.275" x2="-66.04" y2="-31.75" width="0" layer="19" extent="16-16"/>
 <wire x1="-24.765" y1="-2.225" x2="-41.07" y2="-1.27" width="0" layer="19" extent="16-16"/>
 <wire x1="-19.365" y1="1.27" x2="-24.765" y2="-2.225" width="0" layer="19" extent="16-16"/>
@@
 <wire x1="-18.735" y1="-25.4" x2="-16.51" y2="-18.415" width="0" layer="19" extent="16-16"/>
 <wire x1="-18.735" y1="-28.575" x2="-18.735" y2="-25.4" width="0" layer="19" extent="16-16"/>
-<wire x1="-87.37" y1="-22.225" x2="-66.995" y2="-24.13" width="0" layer="19" extent="16-16"/>
 </signal>
 <signal name="N$8">
@@
 <contactref element="R17" pad="1"/>
 <wire x1="-63.5" y1="1.016" x2="-68.58" y2="1.016" width="1.016" layer="16"/>
-<wire x1="-77.155" y1="1.27" x2="-77.155" y2="-1.27" width="0" layer="19" extent="16-16"/>
+<wire x1="-77.155" y1="-1.27" x2="-77.155" y2="1.27" width="0" layer="19" extent="16-16"/>
 <wire x1="-68.58" y1="1.016" x2="-77.155" y2="1.27" width="0" layer="19" extent="16-16"/>
 </signal>
@@
 <wire x1="-89.795" y1="-0.99" x2="-89.795" y2="0.635" width="0.4064" layer="16"/>
 <wire x1="-89.795" y1="0.635" x2="-80.645" y2="0.635" width="0.4064" layer="16"/>
-<wire x1="-79.055" y1="1.27" x2="-80.645" y2="0.635" width="0" layer="19" extent="16-16"/>
+<wire x1="-80.645" y1="0.635" x2="-79.055" y2="1.27" width="0" layer="19" extent="16-16"/>
 </signal>
 <signal name="N$12">
@@
 <contactref element="R9" pad="1"/>
 <contactref element="R10" pad="2"/>
+<wire x1="-17.145" y1="8.255" x2="-13.335" y2="2.855" width="0" layer="19" extent="16-16"/>
 <wire x1="-18.735" y1="11.43" x2="-17.145" y2="8.255" width="0" layer="19" extent="16-16"/>
-<wire x1="-13.335" y1="2.855" x2="-17.145" y2="8.255" width="0" layer="19" extent="16-16"/>
 </signal>
 <signal name="N$26">
@@
 <signal name="N$34">
 <contactref element="R26" pad="1"/>
+<contactref element="VD6" pad="C"/>
+<contactref element="VD5" pad="C"/>
+<wire x1="-159.385" y1="-7.19" x2="-164.465" y2="-7.19" width="0" layer="19" extent="16-16"/>
+<wire x1="-11.43" y1="-19.685" x2="-159.385" y2="-7.19" width="0" layer="19" extent="16-16"/>
 </signal>
 <signal name="+12V">
@@
 <contactref element="R7" pad="2"/>
 <contactref element="OK1" pad="4"/>
-<wire x1="-75.885" y1="-41.275" x2="-81.28" y2="-29.845" width="0" layer="19" extent="16-16"/>
+<wire x1="-81.28" y1="-29.845" x2="-75.885" y2="-41.275" width="0" layer="19" extent="16-16"/>
 <wire x1="-59.69" y1="-42.545" x2="-75.885" y2="-41.275" width="0" layer="19" extent="16-16"/>
 <wire x1="-43.2816" y1="6.985" x2="-59.69" y2="-42.545" width="0" layer="19" extent="16-16"/>
@@
 <contactref element="R33" pad="1"/>
 <contactref element="R37" pad="1"/>
-<wire x1="-88.9" y1="-29.21" x2="-91.44" y2="-29.21" width="0" layer="19" extent="1-1"/>
-<wire x1="-85.09" y1="-32.065" x2="-88.9" y2="-29.21" width="0" layer="19" extent="16-16"/>
+<wire x1="-88.9" y1="-29.21" x2="-88.9" y2="-32.385" width="0" layer="19" extent="1-1"/>
+<wire x1="-91.44" y1="-29.21" x2="-88.9" y2="-29.21" width="0" layer="19" extent="1-1"/>
+<wire x1="-85.09" y1="-32.065" x2="-88.9" y2="-32.385" width="0" layer="19" extent="16-16"/>
 <wire x1="-81.915" y1="-39.055" x2="-85.09" y2="-32.065" width="0" layer="19" extent="16-16"/>
-<wire x1="-88.9" y1="-32.385" x2="-85.09" y2="-32.065" width="0" layer="19" extent="16-16"/>
 </signal>
 <signal name="N$24">
 <contactref element="R34" pad="1"/>
 <contactref element="R33" pad="3"/>
-<wire x1="-94.93" y1="-31.75" x2="-93.98" y2="-29.21" width="0" layer="19" extent="16-16"/>
+<wire x1="-93.98" y1="-29.21" x2="-94.93" y2="-31.75" width="0" layer="19" extent="16-16"/>
 </signal>
 <signal name="V+">
@@
 <contactref element="C20" pad="1"/>
 <contactref element="R34" pad="2"/>
-<wire x1="-85.09" y1="-30.165" x2="-93.03" y2="-31.75" width="0" layer="19" extent="16-16"/>
-<wire x1="-88.9" y1="-29.845" x2="-85.09" y2="-30.165" width="0" layer="19" extent="16-16"/>
+<wire x1="-88.9" y1="-29.845" x2="-93.03" y2="-31.75" width="0" layer="19" extent="16-16"/>
+<wire x1="-85.09" y1="-30.165" x2="-88.9" y2="-29.845" width="0" layer="19" extent="16-16"/>
 </signal>
 <signal name="V-">
 <contactref element="R37" pad="2"/>
 </signal>
+<signal name="N$16">
+<contactref element="R27" pad="2"/>
+<contactref element="TV1B" pad="1"/>
+<contactref element="VD5" pad="A"/>
+<wire x1="-164.465" y1="-14.605" x2="-167.005" y2="-17.78" width="0" layer="19" extent="1-1"/>
+<wire x1="-164.465" y1="-10.59" x2="-164.465" y2="-14.605" width="0" layer="19" extent="16-16"/>
+</signal>
+<signal name="N$25">
+<contactref element="R27" pad="1"/>
+<contactref element="TV1B" pad="3"/>
+<contactref element="VD6" pad="A"/>
+<wire x1="-159.385" y1="-14.605" x2="-156.845" y2="-17.78" width="0" layer="19" extent="1-1"/>
+<wire x1="-159.385" y1="-10.59" x2="-159.385" y2="-14.605" width="0" layer="19" extent="16-16"/>
+</signal>
 </signals>

Commit message: .
Parts:
- removed JP1: (no value), Разъёмы штырьковые 2.54мм:1X01
- added TV2C, TV2D: (no value), Разъёмы штырьковые 2.54мм:1X03
- moved R27 85.2 mm to (-87.0, -58.4)
- moved TV1B 85.2 mm to (-87.0, -55.2)
- moved VD5 85.2 mm to (-89.5, -49.5)
- moved VD6 85.2 mm to (-84.5, -49.5)
- moved D2 22.3 mm to (-111.1, -35.6), turned to 180 degrees
- moved D1 22.1 mm to (-137.2, -35.6), turned to 180 degrees
Connections:
- new net N$35: D1.1, TV2C.1
- new net N$36: D1.3, TV2C.3
- new net N$37: D2.1, TV2D.1
- new net N$38: D2.3, TV2D.3
- new net N$39: D1.2
- new net N$40: D2.2, TV2C.2
- new net N$41: TV2D.2
Routing:
- net N$12: track 15.3 -> 14.7 mm
Changed lines of the file:
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@@
 <circle x="-48.26" y="31.75" radius="3" width="0.5" layer="21"/>
 <dimension x1="-184.785" y1="41.91" x2="-180.34" y2="-34.29" x3="-3.81" y3="3.81" textsize="1.778" layer="21" dtype="vertical"/>
+<circle x="-124.46" y="-5.08" radius="5" width="1.016" layer="21"/>
 </plain>
 <attributes>
@@
 <element name="R7" library="rcl" package="M0805" value="10k" x="-40.64" y="6.35" rot="MR90"/>
 <element name="U$1" library="h" package="H44X32" value="" x="-87.63" y="-6.985" rot="R90"/>
-<element name="JP1" library="Разъёмы штырьковые 2.54мм" package="1X01" value="" x="-12.7" y="13.97"/>
 <element name="VT2" library="m_transistor" package="TO92" value="2N5551" x="-19.685" y="-3.81" rot="R180"/>
 <element name="VT1" library="m_transistor" package="TO92" value="2N5401" x="-19.685" y="9.525"/>
@@
 <element name="R34" library="rcl" package="M0805" value="22k" x="-93.98" y="-31.75" rot="MR180"/>
 <element name="R37" library="rcl" package="M0805" value="47k" x="-81.915" y="-40.005" rot="MR270"/>
-<element name="D1" library="diodes" package="TO247H" value="SBL4020" x="-130.175" y="-56.515"/>
-<element name="D2" library="diodes" package="TO247H" value="SBL4020" x="-103.505" y="-56.515"/>
-<element name="TV1B" library="Разъёмы штырьковые 2.54мм" package="1X03" value="" x="-161.925" y="-14.605"/>
-<element name="VD5" library="diode" package="SOD80C" value="4148" x="-164.465" y="-8.89" rot="MR270"/>
-<element name="VD6" library="diode" package="SOD80C" value="4148" x="-159.385" y="-8.89" rot="MR270"/>
-<element name="R27" library="rcl" package="0207/10" value="240" x="-161.925" y="-17.78" rot="R180"/>
+<element name="D1" library="diodes" package="TO247H" value="SBL4020" x="-137.16" y="-35.56" rot="R180"/>
+<element name="D2" library="diodes" package="TO247H" value="SBL4020" x="-111.125" y="-35.56" rot="R180"/>
+<element name="TV1B" library="Разъёмы штырьковые 2.54мм" package="1X03" value="" x="-86.995" y="-55.245"/>
+<element name="VD5" library="diode" package="SOD80C" value="4148" x="-89.535" y="-49.53" rot="MR270"/>
+<element name="VD6" library="diode" package="SOD80C" value="4148" x="-84.455" y="-49.53" rot="MR270"/>
+<element name="R27" library="rcl" package="0207/10" value="240" x="-86.995" y="-58.42" rot="R180"/>
+<element name="TV2C" library="Разъёмы штырьковые 2.54мм" package="1X03" value="" x="-137.16" y="-20.955" rot="R180"/>
+<element name="TV2D" library="Разъёмы штырьковые 2.54мм" package="1X03" value="" x="-109.22" y="-22.225" rot="R180"/>
 </elements>
 <signals>
@@
 <contactref element="C3" pad="2"/>
 <contactref element="TV1B" pad="2"/>
-<wire x1="-97.79" y1="-18.77" x2="-161.925" y2="-14.605" width="0" layer="19" extent="16-16"/>
-<wire x1="-66.995" y1="-24.13" x2="-87.37" y2="-22.225" width="0" layer="19" extent="16-16"/>
-<wire x1="-66.04" y1="-31.75" x2="-66.995" y2="-24.13" width="0" layer="19" extent="16-16"/>
+<wire x1="-77.785" y1="-41.275" x2="-86.995" y2="-55.245" width="0" layer="19" extent="16-16"/>
+<wire x1="-66.04" y1="-31.75" x2="-77.785" y2="-41.275" width="0" layer="19" extent="16-16"/>
+<wire x1="-66.995" y1="-24.13" x2="-66.04" y2="-31.75" width="0" layer="19" extent="16-16"/>
 <wire x1="-64.135" y1="-11.43" x2="-66.995" y2="-24.13" width="0" layer="19" extent="16-16"/>
 <wire x1="-60.005" y1="1.27" x2="-60.325" y2="-1.27" width="0" layer="19" extent="16-16"/>
@@
 <wire x1="-49.21" y1="15.875" x2="-49.4284" y2="12.065" width="0" layer="19" extent="16-16"/>
 <wire x1="-52.07" y1="23.495" x2="-49.21" y2="15.875" width="0" layer="19" extent="16-16"/>
-<wire x1="-77.785" y1="-41.275" x2="-66.04" y2="-31.75" width="0" layer="19" extent="16-16"/>
 <wire x1="-24.765" y1="-2.225" x2="-41.07" y2="-1.27" width="0" layer="19" extent="16-16"/>
 <wire x1="-19.365" y1="1.27" x2="-24.765" y2="-2.225" width="0" layer="19" extent="16-16"/>
@@
 <wire x1="-18.735" y1="-25.4" x2="-16.51" y2="-18.415" width="0" layer="19" extent="16-16"/>
 <wire x1="-18.735" y1="-28.575" x2="-18.735" y2="-25.4" width="0" layer="19" extent="16-16"/>
+<wire x1="-87.37" y1="-22.225" x2="-66.995" y2="-24.13" width="0" layer="19" extent="16-16"/>
 </signal>
 <signal name="N$8">
@@
 <contactref element="VT11" pad="D"/>
 <wire x1="-92.075" y1="-11.47" x2="-92.075" y2="-7.62" width="1.016" layer="16"/>
-<wire x1="-92.075" y1="-7.62" x2="-85.09" y2="-7.62" width="1.016" layer="16"/>
-<wire x1="-85.09" y1="-7.62" x2="-85.09" y2="-12.065" width="1.016" layer="16"/>
+<wire x1="-92.075" y1="-7.62" x2="-85.725" y2="-7.62" width="1.016" layer="16"/>
+<wire x1="-85.725" y1="-7.62" x2="-85.09" y2="-12.065" width="1.016" layer="16"/>
 <wire x1="-85.09" y1="-12.065" x2="-85.09" y2="-11.47" width="0" layer="19" extent="16-16"/>
 </signal>
@@
 </signal>
 <signal name="N$34">
-<contactref element="R26" pad="1"/>
 <contactref element="VD6" pad="C"/>
 <contactref element="VD5" pad="C"/>
-<wire x1="-159.385" y1="-7.19" x2="-164.465" y2="-7.19" width="0" layer="19" extent="16-16"/>
-<wire x1="-11.43" y1="-19.685" x2="-159.385" y2="-7.19" width="0" layer="19" extent="16-16"/>
+<contactref element="R26" pad="1"/>
+<wire x1="-84.455" y1="-47.83" x2="-89.535" y2="-47.83" width="0" layer="19" extent="16-16"/>
+<wire x1="-11.43" y1="-19.685" x2="-84.455" y2="-47.83" width="0" layer="19" extent="16-16"/>
 </signal>
 <signal name="+12V">
@@
 <contactref element="TV1B" pad="1"/>
 <contactref element="VD5" pad="A"/>
-<wire x1="-164.465" y1="-14.605" x2="-167.005" y2="-17.78" width="0" layer="19" extent="1-1"/>
-<wire x1="-164.465" y1="-10.59" x2="-164.465" y2="-14.605" width="0" layer="19" extent="16-16"/>
+<wire x1="-89.535" y1="-55.245" x2="-92.075" y2="-58.42" width="0" layer="19" extent="1-1"/>
+<wire x1="-89.535" y1="-51.23" x2="-89.535" y2="-55.245" width="0" layer="19" extent="16-16"/>
 </signal>
 <signal name="N$25">
@@
 <contactref element="TV1B" pad="3"/>
 <contactref element="VD6" pad="A"/>
-<wire x1="-159.385" y1="-14.605" x2="-156.845" y2="-17.78" width="0" layer="19" extent="1-1"/>
-<wire x1="-159.385" y1="-10.59" x2="-159.385" y2="-14.605" width="0" layer="19" extent="16-16"/>
+<wire x1="-84.455" y1="-55.245" x2="-81.915" y2="-58.42" width="0" layer="19" extent="1-1"/>
+<wire x1="-84.455" y1="-51.23" x2="-84.455" y2="-55.245" width="0" layer="19" extent="16-16"/>
+</signal>
+<signal name="N$35">
+<contactref element="TV2C" pad="1"/>
+<contactref element="D1" pad="1"/>
+<wire x1="-134.62" y1="-20.955" x2="-131.572" y2="-27.94" width="0" layer="19" extent="1-1"/>
+</signal>
+<signal name="N$36">
+<contactref element="D1" pad="3"/>
+<contactref element="TV2C" pad="3"/>
+<wire x1="-139.7" y1="-20.955" x2="-142.748" y2="-27.94" width="0" layer="19" extent="1-1"/>
+</signal>
+<signal name="N$37">
+<contactref element="D2" pad="1"/>
+<contactref element="TV2D" pad="1"/>
+<wire x1="-106.68" y1="-22.225" x2="-105.537" y2="-27.94" width="0" layer="19" extent="1-1"/>
+</signal>
+<signal name="N$38">
+<contactref element="D2" pad="3"/>
+<contactref element="TV2D" pad="3"/>
+<wire x1="-111.76" y1="-22.225" x2="-116.713" y2="-27.94" width="0" layer="19" extent="1-1"/>
+</signal>
+<signal name="N$39">
+<contactref element="D1" pad="2"/>
+</signal>
+<signal name="N$40">
+<contactref element="D2" pad="2"/>
+<contactref element="TV2C" pad="2"/>
+<wire x1="-111.125" y1="-27.94" x2="-137.16" y2="-20.955" width="0" layer="19" extent="1-1"/>
+</signal>
+<signal name="N$41">
+<contactref element="TV2D" pad="2"/>
 </signal>
 </signals>
