File: B0_DC12_DC51.1.sch (EAGLE design)
At the start: 36 parts, among them Q1 BD140, Q2 BD139, Q3 BD140, Q4 BD139, X1 5566-24, X2 5566-6

Commit message: .
Parts:
- added JP1: (no value), Разъёмы штырьковые 2.54мм:PINHD-1X1
- Q1, Q3: value BD140 -> (none); device transistor-pnp:BD140 -> transistor:-PNP-TO126V
- Q2, Q4: value BD139 -> (none); device transistor-npn:BD139 -> transistor:-NPN-TO126V
Changed lines of the file:
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@@
 <part name="X3" library="con-molex" deviceset="KK-156-4" device=""/>
 <part name="DA3" library="linear" deviceset="TL494*" device="D" technology="B"/>
-<part name="Q1" library="transistor-pnp" deviceset="BD140" device=""/>
-<part name="Q2" library="transistor-npn" deviceset="BD139*" device=""/>
+<part name="Q1" library="transistor" deviceset="*-PNP-" device="TO126V"/>
+<part name="Q2" library="transistor" deviceset="*-NPN-" device="TO126V"/>
 <part name="R6" library="rcl" deviceset="R-EU_" device="M0805" value="470"/>
 <part name="GND1" library="supply1v" deviceset="GND" device=""/>
 <part name="GND2" library="supply1v" deviceset="GND" device=""/>
 <part name="R7" library="rcl" deviceset="R-EU_" device="M0805" value="39"/>
-<part name="Q3" library="transistor-pnp" deviceset="BD140" device=""/>
-<part name="Q4" library="transistor-npn" deviceset="BD139*" device=""/>
+<part name="Q3" library="transistor" deviceset="*-PNP-" device="TO126V"/>
+<part name="Q4" library="transistor" deviceset="*-NPN-" device="TO126V"/>
 <part name="R8" library="rcl" deviceset="R-EU_" device="M0805" value="470"/>
 <part name="GND3" library="supply1v" deviceset="GND" device=""/>
@@
 <part name="D3" library="diode" deviceset="DIODE-" device="SOD80C"/>
 <part name="R14" library="rcl" deviceset="R-EU_" device="M0805" value="10k"/>
+<part name="JP1" library="Разъёмы штырьковые 2.54мм" deviceset="PINHD-1X1" device=""/>
 </parts>
 <sheets>
@@
 <instance part="D3" gate="G$1" x="55.88" y="162.56" rot="R270"/>
 <instance part="R14" gate="G$1" x="76.2" y="175.26"/>
+<instance part="JP1" gate="G$1" x="193.04" y="162.56"/>
 </instances>
 <busses>

Commit message: .
Parts:
- removed Q2: (no value), transistor:-NPN-TO126V
- removed R11: 470, rcl:R-EU_0207/12
- removed R12: 15k, rcl:R-EU_0207/12
- added R15, R16: 470, rcl:R-EU_M0805
- added R17, R18, R19: 22, rcl:R-EU_M0805
- added VT10, VT12, VT9: (no value), m_transistor:MOSFET-N_DPACK
- R1: value 10k -> 15k; device rcl:R-EU_0207/12 -> rcl:R-EU_M0805
- R10: value 100k -> 3k3
- R13: value 220 -> 39; device rcl:R-EU_0207/12 -> rcl:R-EU_M0805
- R14: value 10k -> 39
- R2: value 22 -> 470
- R3: value 22 -> 100k; device rcl:R-EU_M0805 -> rcl:R-EU_R0805
- R4: value 22 -> 220
- R6: value 470 -> 10k; device rcl:R-EU_M0805 -> rcl:R-EU_0207/12
- R7: value 39 -> 10k
- R8: value 470 -> 3k3; device rcl:R-EU_M0805 -> rcl:R-EU_0207/12
- R9: value 39 -> 1k; device rcl:R-EU_M0805 -> rcl:R-EU_0207/12
- VT1: value (none) -> 2N5401; device m_transistor:MOSFET-N_DPACK -> m_transistor:BJT_PNP_TO-92_ECB
- VT2: value (none) -> 2N5551; device m_transistor:MOSFET-N_DPACK -> m_transistor:BJT_NPN_TO-92_ECB
- VT4: device m_transistor:MOSFET-N_DPACK -> transistor:-NPN-TO126V
- renumbered Q1 to VT5, Q3 to VT7, Q4 to VT6, R5 to R20, VT3 to VT11
Connections:
- new net N$23: R10.2, R9.1, VT1.B
- new net N$24: R9.2, VT1.E
- new net N$25: R8.2, VT1.C
- new net N$26: R10.1, VT2.C
- net GND: now also R15.1, R16.1, VT10.S, VT12.S, VT9.S; no longer R12.1, VT1.S, VT2.S, VT4.S
- net N$1: now also R6.2; no longer R1.2
- net N$10: now also R14.2, R16.2; no longer R8.2, R9.2
- net N$11: now also R19.1; no longer R4.1
- net N$12: now also VT12.D; no longer VT4.D
- net N$13: now also R13.1; no longer R7.1
- net N$14: now also R14.1; no longer R9.1
- net N$15: now also VT4.C; no longer Q2.C
- net N$16: now also R7.2; no longer R14.2
- net N$17: now also R19.2; no longer R4.2
- net N$18: now also VT12.G; no longer VT4.G
- net N$19: now also R1.2, R4.1; no longer R12.2, R13.1
- net N$22: now also R2.2, R3.2; no longer R10.2, R11.2
- net N$3: now also VT10.D, VT9.D; no longer VT1.D, VT2.D
- net N$4: now also R17.2, VT9.G; no longer R2.2, VT1.G
- net N$5: now also R18.2, VT10.G; no longer R3.2, VT2.G
- net N$6: now also R3.1; no longer R10.1
- net N$7: now also R2.1, R7.1; no longer R11.1, R14.1
- net N$8: now also R13.2, R15.2, VT4.B; no longer Q2.B, R6.2, R7.2
- net N$9: now also R17.1, R18.1, VT4.E; no longer Q2.E, R2.1, R3.1

Commit message: .
Parts:
- added C10: 100n, rcl:C-EUC0805
- added C20: 407n, rcl:C-EUC0805
- added C9: 220n, rcl:C-EUC0805
- added OK1: PC817, optocoupler:PC817
- added R11: 100k, rcl:R-EU_M0805
- added R12: 10k, rcl:R-EU_M0805
- added R21: 6k8, rcl:R-EU_M0805
- added R22: 33k, rcl:R-EU_M0805
- added R23: 3k3, rcl:R-EU_M0805
- added R24: 220, rcl:R-EU_M0805
- added R25: 2k, rcl:R-EU_M0805
- added R26: 10k, rcl:R-TRIMM3296W
- added R33: 100k, rcl:R-TRIMM3296W
- added R34: 22k, rcl:R-EU_M0805
- added R37: 47k, rcl:R-EU_M0805
- added VD4: 1N5817-B, diode:1N5817-B
- added VT3, VT8: 2N5551, m_transistor:BJT_NPN_TO-92_ECB
- R10, R8, R9: device rcl:R-EU_0207/12 -> rcl:R-EU_M0805
Connections:
- net N$13 renamed CL13
- net N$14 renamed CL14
- removed net N$16: C3.1, C7.-, DA3.OUTC, DA3.VREF, R7.2
- removed net N$25: R8.2, VT1.C
- new net +12V: R21.2
- new net +5VREF: C3.1, C7.-, DA3.OUTC, DA3.VREF, OK1.COL, R12.2, R7.2, R9.2, VT1.E
- new net N$13: D3.A, DA3.+I2, R8.2, VT1.C
- new net N$14: OK1.EMIT, R4.2
- new net N$27: R12.1, VT2.B, VT3.C
- new net N$28: R11.2, VT2.E, VT3.E
- new net N$29: R22.1, R23.2, VT3.B, VT8.C
- new net N$30: C9.1, R21.1, R22.2
- new net N$31: R24.1, VT8.B
- new net N$32: C10.2, R24.2, R25.2, VD4.C
- new net N$33: R26.S, VD4.A
- new net N$34: R26.A
- new net V+: C20.1, OK1.A, R34.2
- new net V-: R37.2
- net GND: now also C10.1, C9.2, R11.1, R23.1, R25.1, R26.E, VT8.E
- net N$21: now also C20.2, OK1.C, R33.A, R33.S, R37.1; no longer D3.A, DA3.+I2
- net N$24: now also R33.E, R34.1; no longer R9.2, VT1.E
Other:
- moved on the sheet: C4, C6, D1, D3, R10, R7, R8, R9, VT1, VT2

Commit message: .
Parts:
- added D4, D6: (no value), diode:DIODE_2SCHOTTKY-SOT93H
Changed lines of the file:
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@@
 <part name="P-1" library="supply1v" deviceset="V-" device=""/>
 <part name="P+6" library="supply1v" deviceset="V+" device=""/>
+<part name="D4" library="diode" deviceset="DIODE_2SCHOTTKY-" device="SOT93H"/>
+<part name="D6" library="diode" deviceset="DIODE_2SCHOTTKY-" device="SOT93H"/>
 </parts>
 <sheets>
@@
 <attribute name="VALUE" x="44.45" y="186.055" size="1.778" layer="96"/>
 </instance>
+<instance part="D4" gate="-B1" x="218.44" y="96.52"/>
+<instance part="D6" gate="-B1" x="215.9" y="134.62"/>
 </instances>
 <busses>

Commit message: .
Parts:
- removed D4, D6: (no value), diode:DIODE_2SCHOTTKY-SOT93H
- added VD1: 2v4, diode:ZENER-DIODESOD80C
- added VD2: 4148, diode:DIODE-SOD80C
- C2: value 470x25v -> 47n; device rcl:CPOL-EUE5-10.5 -> rcl:C-EUC0805
- C3: value 470n -> 820; device rcl:C-EUC0805 -> rcl:C-EU025-025X050
- C4: value 820 -> 220n; device rcl:C-EU025-025X050 -> rcl:C-EUC0805
- C5: value 47n -> 470x25v; device rcl:C-EUC0805 -> rcl:CPOL-EUE5-10.5
- C6: value 220n -> 47x25v; device rcl:C-EUC0805 -> rcl:CPOL-EUE5-10.5
- C7: value 47x25v -> 470n; device rcl:CPOL-EUE5-10.5 -> rcl:C-EUC0805
- D1: value (none) -> SBL4020; device diode:ZENER-DIODESOD80C -> diodes:SCHOTTKY_DUALTO247H
- D2: value (none) -> SBL4020; device diode:DIODE-SOD80C -> diodes:SCHOTTKY_DUALTO247H
- VD3: value (none) -> 4148
- renumbered D3 to VD3
Connections:
- net +5VREF: now also C6.-, C7.1; no longer C3.1, C7.-
- net GND: now also C5.-, C7.2, VD1.A, VD2.A; no longer C2.-, C6.2, D1.A, D2.A
- net N$15: now also C4.1, C5.+; no longer C1.1, C2.+
- net N$2: now also C3.1; no longer C4.1
- net N$20: now also C6.+, VD2.C; no longer C7.+, D2.C
- net N$22: now also C2.1; no longer C5.1
- net N$6: now also C2.2; no longer C5.2
- net N$7: now also C1.1, VD1.C; no longer C6.1, D1.C
Other:
- moved on the sheet: C1, C3, C4, R1, R2

Commit message: 2
Parts:
- added R27: 240, rcl:R-EU_0207/10
- added TV1B: (no value), Разъёмы штырьковые 2.54мм:PINHD-1X3
- added VD5, VD6: 4148, diode:DIODE-SOD80C
Connections:
- new net N$16: R27.2, TV1B.1, VD5.A
- new net N$25: R27.1, TV1B.3, VD6.A
- net GND: now also TV1B.2
- net N$34: now also VD5.C, VD6.C
Changed lines of the file:
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@@
 <part name="D1" library="diodes" deviceset="SCHOTTKY_DUAL" device="TO247H" value="SBL4020"/>
 <part name="D2" library="diodes" deviceset="SCHOTTKY_DUAL" device="TO247H" value="SBL4020"/>
+<part name="TV1B" library="Разъёмы штырьковые 2.54мм" deviceset="PINHD-1X3" device=""/>
+<part name="VD5" library="diode" deviceset="DIODE-" device="SOD80C" value="4148"/>
+<part name="VD6" library="diode" deviceset="DIODE-" device="SOD80C" value="4148"/>
+<part name="GND10" library="supply1v" deviceset="GND" device=""/>
+<part name="R27" library="rcl" deviceset="R-EU_" device="0207/10" value="240"/>
 </parts>
 <sheets>
@@
 <instance part="D1" gate="G$1" x="213.36" y="121.92"/>
 <instance part="D2" gate="G$1" x="208.28" y="106.68"/>
+<instance part="TV1B" gate="A" x="116.84" y="43.18"/>
+<instance part="VD5" gate="G$1" x="93.98" y="50.8" smashed="yes" rot="MR0">
+<attribute name="NAME" x="91.44" y="47.7774" size="1.778" layer="95" rot="MR180"/>
+<attribute name="VALUE" x="91.44" y="45.4914" size="1.778" layer="96" rot="MR180"/>
+</instance>
+<instance part="VD6" gate="G$1" x="93.98" y="35.56" smashed="yes" rot="MR0">
+<attribute name="NAME" x="91.44" y="42.6974" size="1.778" layer="95" rot="MR180"/>
+<attribute name="VALUE" x="91.44" y="40.4114" size="1.778" layer="96" rot="MR180"/>
+</instance>
+<instance part="GND10" gate="1" x="104.14" y="43.18" rot="R270"/>
+<instance part="R27" gate="G$1" x="99.06" y="43.18" smashed="yes" rot="R90">
+<attribute name="NAME" x="100.33" y="47.2186" size="1.778" layer="95"/>
+<attribute name="VALUE" x="100.33" y="37.338" size="1.778" layer="96"/>
+</instance>
 </instances>
 <busses>
@@
 <pinref part="GND20" gate="1" pin="GND"/>
 <wire x1="63.5" y1="66.04" x2="63.5" y2="63.5" width="0.1524" layer="91"/>
+</segment>
+<segment>
+<pinref part="GND10" gate="1" pin="GND"/>
+<pinref part="TV1B" gate="A" pin="2"/>
+<wire x1="106.68" y1="43.18" x2="114.3" y2="43.18" width="0.1524" layer="91"/>
 </segment>
 </net>
@@
 <pinref part="R26" gate="G$1" pin="A"/>
 <wire x1="78.74" y1="45.72" x2="78.74" y2="43.18" width="0.1524" layer="91"/>
+<pinref part="VD6" gate="G$1" pin="C"/>
+<wire x1="91.44" y1="35.56" x2="88.9" y2="35.56" width="0.1524" layer="91"/>
+<wire x1="88.9" y1="35.56" x2="88.9" y2="43.18" width="0.1524" layer="91"/>
+<pinref part="VD5" gate="G$1" pin="C"/>
+<wire x1="88.9" y1="43.18" x2="88.9" y2="50.8" width="0.1524" layer="91"/>
+<wire x1="88.9" y1="50.8" x2="91.44" y2="50.8" width="0.1524" layer="91"/>
+<wire x1="78.74" y1="43.18" x2="88.9" y2="43.18" width="0.1524" layer="91"/>
+<junction x="88.9" y="43.18"/>
 </segment>
 </net>
@@
 </segment>
 </net>
+<net name="N$16" class="0">
+<segment>
+<pinref part="R27" gate="G$1" pin="2"/>
+<wire x1="99.06" y1="48.26" x2="99.06" y2="50.8" width="0.1524" layer="91"/>
+<wire x1="99.06" y1="50.8" x2="106.68" y2="50.8" width="0.1524" layer="91"/>
+<wire x1="106.68" y1="50.8" x2="106.68" y2="45.72" width="0.1524" layer="91"/>
+<pinref part="TV1B" gate="A" pin="1"/>
+<wire x1="106.68" y1="45.72" x2="114.3" y2="45.72" width="0.1524" layer="91"/>
+<pinref part="VD5" gate="G$1" pin="A"/>
+<wire x1="96.52" y1="50.8" x2="99.06" y2="50.8" width="0.1524" layer="91"/>
+<junction x="99.06" y="50.8"/>
+</segment>
+</net>
+<net name="N$25" class="0">
+<segment>
+<pinref part="R27" gate="G$1" pin="1"/>
+<wire x1="99.06" y1="38.1" x2="99.06" y2="35.56" width="0.1524" layer="91"/>
+<wire x1="99.06" y1="35.56" x2="106.68" y2="35.56" width="0.1524" layer="91"/>
+<wire x1="106.68" y1="35.56" x2="106.68" y2="40.64" width="0.1524" layer="91"/>
+<pinref part="TV1B" gate="A" pin="3"/>
+<wire x1="106.68" y1="40.64" x2="114.3" y2="40.64" width="0.1524" layer="91"/>
+<pinref part="VD6" gate="G$1" pin="A"/>
+<wire x1="96.52" y1="35.56" x2="99.06" y2="35.56" width="0.1524" layer="91"/>
+<junction x="99.06" y="35.56"/>
+</segment>
+</net>

Commit message: .
Parts:
- removed JP1: (no value), Разъёмы штырьковые 2.54мм:PINHD-1X1
- added TV2C, TV2D: (no value), Разъёмы штырьковые 2.54мм:PINHD-1X3
Connections:
- new net N$35: D1.A1, TV2C.1
- new net N$36: D1.A2, TV2C.3
- new net N$37: D2.A1, TV2D.1
- new net N$38: D2.A2, TV2D.3
- new net N$39: D1.C
- new net N$40: D2.C, TV2C.2
- new net N$41: TV2D.2
Other:
- moved on the sheet: D1, D2, R26, R27, TV1B, VD5, VD6
